File: hardware/PCB/Smartwatch.kicad_sch (KiCad schematic)
At the start: 142 parts, among them J1 USB_B_Micro, J2 BATT, J3 Conn_01x15, J5 PROGRAM, Q1 DMG1012T, SW1 SW_Push, SW2 SW_Push, SW3 SW_Push, U1 RV1103, U2 EA3036C, U3 MCP73871, U4 W25N01KVZEIR, U5 ATtiny10-TS, U6 RTL8723BS, Y1 24MHz

Commit message: PCB rev.B completed
Parts:
- removed AE1: 2.4Ghz, ildus_footprints:2.4Ghz_TE_Antenna, symbol ildus_custom_lib:Ant_chip_2_4Ghz
- removed C22: 100nF, Capacitor_SMD:C_0201_0603Metric, symbol Device:C
- removed C59: 100pF, Capacitor_SMD:C_0201_0603Metric, symbol Device:C
- removed U5: ATtiny10-TS, Package_TO_SOT_SMD:SOT-23-6, symbol MCU_Microchip_ATtiny:ATtiny10-TS
- added AE1: Antenna, ildus_footprints:5320_2.4Ghz_antenna, symbol Device:Antenna
- added BZ1: Buzzer, ildus_footprints:MLT-5020_buzzer, symbol Device:Buzzer
- added C60, C61: 18pF, Capacitor_SMD:C_0201_0603Metric, symbol Device:C
- added D7: STAT, LED_SMD:LED_0402_1005Metric_Pad0.77x0.64mm_HandSolder, symbol Device:LED
- added D8: BAT30F4, Diode_SMD:D_0201_0603Metric, symbol Device:D_Small
- added Q2, Q3: DMG1012T, Package_TO_SOT_SMD:SOT-523, symbol Transistor_FET:DMG1012T
- added R44, R47: 1K, Resistor_SMD:R_0201_0603Metric, symbol Device:R_US
- added R45: 0R, Resistor_SMD:R_0402_1005Metric_Pad0.72x0.64mm_HandSolder, symbol Device:R_US
- added R46: 0R (DNP), Resistor_SMD:R_0402_1005Metric_Pad0.72x0.64mm_HandSolder, symbol Device:R_US
- added R48, R52: 10K, Resistor_SMD:R_0201_0603Metric, symbol Device:R_US
- added R49, R51: 100, Resistor_SMD:R_0201_0603Metric, symbol Device:R_US
- added R50: 100R, Resistor_SMD:R_0201_0603Metric, symbol Device:R_US
- added TP12: TestPoint, ildus_footprints:TP, symbol Connector:TestPoint
- added U5: TXS0102DQE, Package_SON:X2SON-8_1.4x1mm_P0.35mm, symbol Logic_LevelTranslator:TXS0102DQE
- added U7: ATtiny816-M, Package_DFN_QFN:VQFN-20-1EP_3x3mm_P0.4mm_EP1.7x1.7mm, symbol MCU_Microchip_ATtiny:ATtiny816-M
- added U8: QMI8658, Package_LGA:Bosch_LGA-14_3x2.5mm_P0.5mm, symbol ildus_custom_lib:QMI8658
- added Y2: 32.768Khz, Crystal:Crystal_SMD_2012-2Pin_2.0x1.2mm, symbol Device:Crystal
- D1: value LED -> PG; footprint LED_SMD:LED_0201_0603Metric -> LED_SMD:LED_0402_1005Metric_Pad0.77x0.64mm_HandSolder
- D2: value LED -> CHRG; footprint LED_SMD:LED_0201_0603Metric -> LED_SMD:LED_0402_1005Metric_Pad0.77x0.64mm_HandSolder
- D3: value LED -> DONE; footprint LED_SMD:LED_0201_0603Metric -> LED_SMD:LED_0402_1005Metric_Pad0.77x0.64mm_HandSolder
- D4, D5: footprint LED_SMD:LED_0201_0603Metric -> LED_SMD:LED_0402_1005Metric
- R10, R11, R12: value 1K -> 100R
- R22, R23: value 4K7 -> 47K
- R29: value 10K -> 100
- R41: value 47K(NC) -> 2K
- R43: value 10K -> 47K
Connections:
- net +3V3: now also C42.1, R22.1, R23.2, R43.2; no longer C42.2
- net GND: now also C40.1, C42.2, J5.2 (Pin_2), C60.1, C61.2, D7.1 (K), Q2.2 (S), R48.1, R50.2, U5.4 (GND), U7.21 (GND), U7.3 (GND), U8.1 (SDO/SA0), U8.6 (GND), U8.7 (GND); no longer C40.2, C42.1, J5.6 (Pin_6), R41.2, U3.4 (PROG2)
- net I2C4_SCL: now also U5.7 (B1), U8.13 (SCL); no longer R22.1
- net I2C4_SDA: now also U5.6 (B2), U8.14 (SDA); no longer R23.1
- net LCD_BCKL: now also U1.42 (PWM1_M0_PWR_CTRL_M0G_PIO0_A4_d); no longer U1.56 (UART3_RX_M1_UART5_CTS_M1_PWM10_M2__GPIO1_D1_d)
- net LCD_DC: now also U1.62 (I2C4_SDA_M1_SDIO_CMD_M1_SPI0_MISO_M0_PWM6_M2__GPIO1_C3_d); no longer U1.53 (UART4_CTS_M1_PWM11_IR_M1__GPIO1_C7_d)
- net PWR_KEY: now also J5.3 (Pin_3), U7.16 (PC1); no longer J5.4 (Pin_4)
- net VBAT_ADC: now also U7.10 (PB4); no longer U1.15 (PWM1_M1_SARADC_IN1_GPIO4_C1_z)
- net VBUS: now also R41.2, R46.1; no longer D1.2 (A), D2.2 (A), D3.2 (A)
- net VCC_1V8: now also D1.2 (A), D2.2 (A), D3.2 (A), U5.8 (VCCB), U8.12 (CS), U8.2 (SDx), U8.3 (SCx), U8.5 (VDDIO), U8.8 (VDD); no longer R22.2, R23.2, R43.2
- net WIFI_EN: now also U1.2 (GPIO3_C5_d), R51.1; no longer U1.8 (SDMMC_DET__GPIO3_A1_u), U6.12 (WL_DSI#), U6.13 (WL_HOST_WAKE)
- net BT_EN: now reaches R42.1, U6.34 (BT_DIS#)
- net BT_EN: now also U1.82 (LVDS_RX_D1N_MIPI_CSI_RX_D1N__GPI3_B6_d); no longer R41.1
- net CHRG: now reaches R11.1, U3.8 (STAT1/~{LBO})
- net CHRG: now also U1.84 (LVDS_RX_CLK0N_MIPI_CSI_RX_CLK0N__GPI3_C0_d)
- net at U1.22 (CODEC_VCM): now also C40.2; no longer C40.1
- net UART4_TX: now reaches TP8.1, U1.60 (SDIO_D2_M1_UART4_TX_M1_PWM9_M1__GPIO1_C5_d)
- net UART4_TX: now also U6.43 (UART_IN)
- net at D6.1 (K), J5.1 (Pin_1): now also U5.1 (VCCA), U7.4 (VCC)
- net UART4_CTS: now reaches U6.41 (UART_RTS)
- net UART4_CTS: now also U1.53 (UART4_CTS_M1_PWM11_IR_M1__GPIO1_C7_d)
- net UART4_RX: now reaches U6.42 (UART_OUT)
- net UART4_RX: now also TP9.1, U1.61 (SDIO_D3_M1_UART4_RX_M1_PWM8_M1__GPIO1_C4_d)
- net UART4_RTS: now reaches U6.44 (UART_CTS)
- net UART4_RTS: now also U1.52 (UART4_RTS_M1_PWM10_M1__GPIO1_C6_d)
- net at U6.6 (BT_WAKE): now also R22.2
- net DONE: now reaches R12.1, U3.7 (STAT2)
- net DONE: now also U1.85 (LVDS_RX_CLK0P_MIPI_CSI_RX_CLK0P__GPI3_C1_d)
- net at C58.2: now also AE1.1 (A)
- net READ_REQ: now reaches U1.1 (MIPI_CLK0_OUT__GPIO3_C4_d)
- net READ_REQ: now also J5.6 (Pin_6), U7.7 (PA6)
- net QMI_INT2: now reaches U1.86 (LVDS_RX_D0N_MIPI_CSI_RX_D0N__GPI3_C2_d)
- net QMI_INT2: now also U8.9 (INT2)
- net QMI_INT1: now reaches U1.87 (LVDS_RX_D0P_MIPI_CSI_RX_D0P__GPI3_C3_d)
- net QMI_INT1: now also U8.4 (INT1)
- net LCD_RES renamed LCD_RST
- net LCD_RST: now also U1.56 (UART3_RX_M1_UART5_CTS_M1_PWM10_M2__GPIO1_D1_d); no longer U1.52 (UART4_RTS_M1_PWM10_M1__GPIO1_C6_d)
- removed net PMIC_EN: J5.2 (Pin_2), U2.18 (EN3), U2.8 (EN2), U2.9 (EN1)
- removed net PWR_RX_NOTIFY: J5.3 (Pin_3), R43.1, U1.81 (LVDS_RX_D2P_MIPI_CSI_RX_D2P__GPI3_B5_d)
- net PWR_TX_NOTIFY renamed UART_TXD
- net UART_TXD: now also U7.20 (PA1); no longer U1.42 (PWM1_M0_PWR_CTRL_M0G_PIO0_A4_d)
- net VCC_CHRG renamed VCC_MCP
- net VCC_MCP: now also R45.2, R46.2, R49.2; no longer C37.1, TP1.1, U3.1 (OUT), U3.20 (OUT)
- new net: Q3.1 (G), R51.2, R52.2
- new net: Q3.2 (S), R52.1
- new net: Q3.3 (D), R23.1, U6.12 (WL_DSI#)
- new net: C61.1, U7.11 (PB3), Y2.1
- new net: C60.2, U7.12 (PB2), Y2.2
- new net: TP12.1, U1.15 (PWM1_M1_SARADC_IN1_GPIO4_C1_z)
- new net: R44.1, U7.15 (PC0)
- new net: D7.2 (A), R44.2
- new net: C37.1, R45.1, TP1.1, U3.1 (OUT), U3.20 (OUT)
- new net: BZ1.1 (+), D8.1 (K), R49.1
- new net: R41.1, U3.4 (PROG2)
- new net: U5.2 (A1), U7.14 (PB0)
- new net: U5.3 (A2), U7.13 (PB1)
- new net: U5.5 (OE), U7.8 (PA7)
- new net: R43.1, U6.13 (WL_HOST_WAKE)
- new net: Q2.1 (G), R47.2, R48.2
- new net: BZ1.2 (-), D8.2 (A), Q2.3 (D)
- new net: R50.1, U1.8 (SDMMC_DET__GPIO3_A1_u)
- new net BUZZER: R47.1, U7.6 (PA5)
- new net PMIC_EN1: U2.9 (EN1), U7.1 (PA2)
- new net PMIC_EN2: U2.8 (EN2), U7.2 (PA3)
- new net PMIC_EN3: U2.18 (EN3), U7.17 (PC2)
- new net UDPI: J5.4 (Pin_4), U7.19 (~{RESET}/PA0)
- no-connect marks 32 -> 25
Other:
- note added: "BUZZER"
- note added: "DEBUG"
- note added: "FILTERS"
- note added: "MEMS"
- note added: "POWER CONTROL & RTC"
- note added: "WIFI & BLUETOOTH"
- note removed: ""CHARGE""
- note removed: ""DONE""
- note removed: ""PWR""
- note removed: "POWER CONTROL"
- note removed: "TODO: -CHECK WAKEUP LINE (GPIO1_A) PWR_TX_NOTIFY -ADD BLUETOOTH -ADD WIFI -RENAME VCC5V0_SYS TO XXX -change 1uf to 0201 -add RTC"
- note removed: "WIFI"
- moved on the sheet: C1, C10, C11, C12, C13, C14, C15, C16, C17, C18, C19, C2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
